File: fuente_flyback.kicad_sch (KiCad schematic)
At the start: 12 parts, among them T1 Transformer_1P_1S

Commit message: make some simulations
Parts:
- added R?: 10, symbol Device:R
Connections:
- net MOSFET_CTRL: now also R?.1; no longer Q?.2 (G)
- new net: Q?.2 (G), R?.2
Changed lines of the file:
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@@
+    (stroke (width 0) (type solid) (color 0 0 0 0))
+  )
+  (wire (pts (xy 123.825 94.615) (xy 125.095 94.615))
     (stroke (width 0) (type solid) (color 0 0 0 0))
   )
@@
     (stroke (width 0) (type solid) (color 0 0 0 0))
   )
-  (wire (pts (xy 130.81 94.615) (xy 133.35 94.615))
+  (wire (pts (xy 132.715 94.615) (xy 133.35 94.615))
     (stroke (width 0) (type solid) (color 0 0 0 0))
   )
@@
     )
   )
-  (global_label "MOSFET_CTRL" (shape input) (at 130.81 94.615 180) (fields_autoplaced)
+  (global_label "MOSFET_CTRL" (shape input) (at 123.825 94.615 180) (fields_autoplaced)
     (effects (font (size 1.27 1.27)) (justify right))
-    (property "Intersheet References" "${INTERSHEET_REFS}" (id 0) (at 115.6969 94.5356 0)
+    (property "Intersheet References" "${INTERSHEET_REFS}" (id 0) (at 108.7119 94.5356 0)
       (effects (font (size 1.27 1.27)) (justify right) hide)
     )
@@
     (pin "2")
   )
+  (symbol (lib_id "Device:R") (at 128.905 94.615 90) (unit 1)
+    (in_bom yes) (on_board yes) (fields_autoplaced)
+    (property "Reference" "R?" (id 0) (at 128.905 90.1658 90))
+    (property "Value" "10" (id 1) (at 128.905 92.4645 90))
+    (property "Footprint" "" (id 2) (at 128.905 96.393 90)
+      (effects (font (size 1.27 1.27)) hide)
+    )
+    (property "Datasheet" "~" (id 3) (at 128.905 94.615 0)
+      (effects (font (size 1.27 1.27)) hide)
+    )
+    (pin "1")
+    (pin "2")
+  )
   (symbol (lib_id "Connector:Conn_01x02_Female") (at 43.18 54.61 180) (unit 1)
     (in_bom yes) (on_board yes)
@@
       (reference "Q?") (unit 1) (value "Q_NMOS_DGS") (footprint "")
     )
+    (path "/642f885e-bf43-4313-a55c-85a8d40e226d"
+      (reference "R?") (unit 1) (value "10") (footprint "")
+    )
     (path "/b0d8b8d3-3c8a-48ef-8a5b-8f060bc848a9"
       (reference "T1") (unit 1) (value "Transformer_1P_1S") (footprint "Transformer_THT:Transformer_NF_ETAL_P3356")
@@
     )
     (path "/051008e0-21d7-4cb8-a579-83f0279b9efb/83fbb457-623f-4695-8e88-2a124690cefd"
-      (reference "C?") (unit 1) (value "100n") (footprint "")
+      (reference "C31") (unit 1) (value "1.5n") (footprint "")
+    )
+    (path "/051008e0-21d7-4cb8-a579-83f0279b9efb/627b689f-bb7c-4620-8ae7-bdc4f112948d"
+      (reference "D31") (unit 1) (value "1N4148") (footprint "Diode_THT:D_DO-35_SOD27_P7.62mm_Horizontal")
     )
     (path "/051008e0-21d7-4cb8-a579-83f0279b9efb/3b546506-e4be-4bf9-899a-1654a58ac16a"
-      (reference "D?") (unit 1) (value "1N4148") (footprint "Diode_THT:D_DO-35_SOD27_P7.62mm_Horizontal")
-    )
-    (path "/051008e0-21d7-4cb8-a579-83f0279b9efb/627b689f-bb7c-4620-8ae7-bdc4f112948d"
-      (reference "D?") (unit 1) (value "1N4148") (footprint "Diode_THT:D_DO-35_SOD27_P7.62mm_Horizontal")
+      (reference "D32") (unit 1) (value "1N4148") (footprint "Diode_THT:D_DO-35_SOD27_P7.62mm_Horizontal")
+    )
+    (path "/051008e0-21d7-4cb8-a579-83f0279b9efb/e8252336-51a8-4bea-8920-cce66aa0eb88"
+      (reference "D33") (unit 1) (value "1N4148") (footprint "Diode_THT:D_DO-35_SOD27_P7.62mm_Horizontal")
     )
     (path "/051008e0-21d7-4cb8-a579-83f0279b9efb/755e20c0-5ce5-4733-bdac-dd2777514a0a"
-      (reference "D?") (unit 1) (value "1N4148") (footprint "Diode_THT:D_DO-35_SOD27_P7.62mm_Horizontal")
+      (reference "D34") (unit 1) (value "1N4148") (footprint "Diode_THT:D_DO-35_SOD27_P7.62mm_Horizontal")
+    )
+    (path "/051008e0-21d7-4cb8-a579-83f0279b9efb/e149cf92-9b3c-4143-9640-abbb5820f5ed"
+      (reference "D35") (unit 1) (value "1N4148") (footprint "Diode_THT:D_DO-35_SOD27_P7.62mm_Horizontal")
+    )
+    (path "/051008e0-21d7-4cb8-a579-83f0279b9efb/97c7d7d3-333e-48a4-a5dc-b02451811911"
+      (reference "D36") (unit 1) (value "1N4148") (footprint "Diode_THT:D_DO-35_SOD27_P7.62mm_Horizontal")
+    )
+    (path "/051008e0-21d7-4cb8-a579-83f0279b9efb/8cd4e952-4827-4c48-9c0a-53b22888d242"
+      (reference "D37") (unit 1) (value "1N4148") (footprint "Diode_THT:D_DO-35_SOD27_P7.62mm_Horizontal")
     )
     (path "/051008e0-21d7-4cb8-a579-83f0279b9efb/7d1aabbc-9dbc-4082-a153-970a2a8ee561"
-      (reference "D?") (unit 1) (value "1N4148") (footprint "Diode_THT:D_DO-35_SOD27_P7.62mm_Horizontal")
-    )
-    (path "/051008e0-21d7-4cb8-a579-83f0279b9efb/8cd4e952-4827-4c48-9c0a-53b22888d242"
-      (reference "D?") (unit 1) (value "1N4148") (footprint "Diode_THT:D_DO-35_SOD27_P7.62mm_Horizontal")
-    )
-    (path "/051008e0-21d7-4cb8-a579-83f0279b9efb/97c7d7d3-333e-48a4-a5dc-b02451811911"
-      (reference "D?") (unit 1) (value "1N4148") (footprint "Diode_THT:D_DO-35_SOD27_P7.62mm_Horizontal")
-    )
-    (path "/051008e0-21d7-4cb8-a579-83f0279b9efb/e149cf92-9b3c-4143-9640-abbb5820f5ed"
-      (reference "D?") (unit 1) (value "1N4148") (footprint "Diode_THT:D_DO-35_SOD27_P7.62mm_Horizontal")
-    )
-    (path "/051008e0-21d7-4cb8-a579-83f0279b9efb/e8252336-51a8-4bea-8920-cce66aa0eb88"
-      (reference "D?") (unit 1) (value "1N4148") (footprint "Diode_THT:D_DO-35_SOD27_P7.62mm_Horizontal")
+      (reference "D38") (unit 1) (value "1N4148") (footprint "Diode_THT:D_DO-35_SOD27_P7.62mm_Horizontal")
+    )
+    (path "/051008e0-21d7-4cb8-a579-83f0279b9efb/8cd3267d-b4e4-4d8d-9e87-d4fc072a03a7"
+      (reference "Q31") (unit 1) (value "MMBT3906") (footprint "Package_TO_SOT_SMD:SOT-23")
     )
     (path "/051008e0-21d7-4cb8-a579-83f0279b9efb/727cf34d-140c-48b6-9936-d91d5a57cf44"
-      (reference "Q?") (unit 1) (value "MMBT3904") (footprint "Package_TO_SOT_SMD:SOT-23")
-    )
-    (path "/051008e0-21d7-4cb8-a579-83f0279b9efb/8cd3267d-b4e4-4d8d-9e87-d4fc072a03a7"
-      (reference "Q?") (unit 1) (value "MMBT3906") (footprint "Package_TO_SOT_SMD:SOT-23")
+      (reference "Q32") (unit 1) (value "MMBT3904") (footprint "Package_TO_SOT_SMD:SOT-23")
+    )
+    (path "/051008e0-21d7-4cb8-a579-83f0279b9efb/44e6a983-74c4-4b8f-8701-f0cb759166a3"
+      (reference "R31") (unit 1) (value "1k") (footprint "")
+    )
+    (path "/051008e0-21d7-4cb8-a579-83f0279b9efb/60d820d1-5edd-4063-916b-1c73eebed3c3"
+      (reference "R32") (unit 1) (value "330") (footprint "")
+    )
+    (path "/051008e0-21d7-4cb8-a579-83f0279b9efb/8c7b13d2-5b6f-4d20-9fce-36e7d761ac93"
+      (reference "R34") (unit 1) (value "2k") (footprint "")
+    )
+    (path "/051008e0-21d7-4cb8-a579-83f0279b9efb/575e4595-5c5d-49ef-897f-6e1e5b82d107"
+      (reference "R35") (unit 1) (value "3k") (footprint "")
+    )
+    (path "/051008e0-21d7-4cb8-a579-83f0279b9efb/6de1a8eb-5323-4076-a723-36db8959b763"
+      (reference "R36") (unit 1) (value "9k") (footprint "")
+    )
+    (path "/051008e0-21d7-4cb8-a579-83f0279b9efb/18d5ae91-676b-404b-ac3a-8063f77c0e47"
+      (reference "R37") (unit 1) (value "9k") (footprint "")
     )
     (path "/051008e0-21d7-4cb8-a579-83f0279b9efb/093a3a24-d61f-4a29-8c3e-60d6075cf876"
       (reference "R?") (unit 1) (value "2k") (footprint "")
     )
-    (path "/051008e0-21d7-4cb8-a579-83f0279b9efb/18d5ae91-676b-404b-ac3a-8063f77c0e47"
-      (reference "R?") (unit 1) (value "3.9k") (footprint "")
-    )
-    (path "/051008e0-21d7-4cb8-a579-83f0279b9efb/44e6a983-74c4-4b8f-8701-f0cb759166a3"
-      (reference "R?") (unit 1) (value "1k") (footprint "")
-    )
-    (path "/051008e0-21d7-4cb8-a579-83f0279b9efb/575e4595-5c5d-49ef-897f-6e1e5b82d107"
-      (reference "R?") (unit 1) (value "3.9k") (footprint "")
-    )
-    (path "/051008e0-21d7-4cb8-a579-83f0279b9efb/60d820d1-5edd-4063-916b-1c73eebed3c3"
-      (reference "R?") (unit 1) (value "R") (footprint "")
-    )
-    (path "/051008e0-21d7-4cb8-a579-83f0279b9efb/6de1a8eb-5323-4076-a723-36db8959b763"
-      (reference "R?") (unit 1) (value "3.9k") (footprint "")
-    )
-    (path "/051008e0-21d7-4cb8-a579-83f0279b9efb/8c7b13d2-5b6f-4d20-9fce-36e7d761ac93"
-      (reference "R?") (unit 1) (value "2k") (footprint "")
-    )
     (path "/051008e0-21d7-4cb8-a579-83f0279b9efb/d7eae77d-540b-4c0e-aaf7-5c58eca2eb83"
-      (reference "R?") (unit 1) (value "R") (footprint "")
+      (reference "R?") (unit 1) (value "330") (footprint "")
     )
     (path "/051008e0-21d7-4cb8-a579-83f0279b9efb/c2d9c4bd-46f7-4b4c-b31b-3c0e12ff4177"
@@
     )
     (path "/051008e0-21d7-4cb8-a579-83f0279b9efb/4ada94f8-9250-41d8-81df-1a0b39db40ac"
-      (reference "U?") (unit 1) (value "LM319") (footprint "")
+      (reference "U31") (unit 1) (value "LM319") (footprint "")
     )
     (path "/051008e0-21d7-4cb8-a579-83f0279b9efb/b9522152-f8fc-4d33-ab52-f9cfa7a8d6f6"
-      (reference "U?") (unit 1) (value "LM319") (footprint "")
-    )
-  )
+      (reference "U31") (unit 2) (value "LM319") (footprint "")
+    )
+  )
