File: triangular_signal.kicad_sch (KiCad schematic)
At the start: 23 parts

Commit message: make some simulations
Parts:
- C31: renamed from C?; value 100n -> 1.5n
- R32: renamed from R?; value R -> 330
- R35: renamed from R?; value 3.9k -> 3k
- R36, R37: renamed from R?; value 3.9k -> 9k
- R?: value R -> 330
- gave numbers to parts that had none: 13
Connections:
- net FEEDBACK_SIGNAL: now also U31.10 (-); no longer U31.5 (-)
- net GNDPWR: now also U31.8 (Gnd); no longer U31.3 (Gnd)
- net MOSFET_CTRL: now also U31.7; no longer U31.12
- net at C31.1, D37.1 (K), D38.2 (A)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: now also U31.9 (+); no longer U31.4 (+)
Changed lines of the file:
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@@
   (junction (at 189.23 103.505) (diameter 1.016) (color 0 0 0 0))
   (junction (at 193.04 136.525) (diameter 1.016) (color 0 0 0 0))
+  (junction (at 201.93 103.505) (diameter 1.016) (color 0 0 0 0))
   (wire (pts (xy 34.29 149.225) (xy 39.37 149.225))
     (stroke (width 0) (type solid) (color 0 0 0 0))
@@
     (stroke (width 0) (type solid) (color 0 0 0 0))
   )
+  (wire (pts (xy 201.93 103.505) (xy 207.645 103.505))
+    (stroke (width 0) (type solid) (color 0 0 0 0))
+  )
   (wire (pts (xy 203.2 136.525) (xy 193.04 136.525))
     (stroke (width 0) (type solid) (color 0 0 0 0))
   )
-  (label "sw_control" (at 109.22 106.045 0)
-    (effects (font (size 1.27 1.27)) (justify left bottom))
-  )
-  (label "sw_control" (at 194.31 103.505 0)
-    (effects (font (size 1.27 1.27)) (justify left bottom))
+  (global_label "sw_control" (shape input) (at 107.95 106.045 180) (fields_autoplaced)
+    (effects (font (size 1.27 1.27)) (justify right))
+    (property "Intersheet References" "${INTERSHEET_REFS}" (id 0) (at 95.4979 105.9656 0)
+      (effects (font (size 1.27 1.27)) (justify right) hide)
+    )
+  )
+  (global_label "sw_control" (shape input) (at 207.645 103.505 0) (fields_autoplaced)
+    (effects (font (size 1.27 1.27)) (justify left))
+    (property "Intersheet References" "${INTERSHEET_REFS}" (id 0) (at 220.0971 103.4256 0)
+      (effects (font (size 1.27 1.27)) (justify left) hide)
+    )
   )
   (hierarchical_label "PWRGND" (shape input) (at 34.29 149.225 180)
@@
   (symbol (lib_id "Device:R") (at 72.39 106.045 0) (unit 1)
     (in_bom yes) (on_board yes)
-    (property "Reference" "R?" (id 0) (at 74.168 104.8766 0)
+    (property "Reference" "R31" (id 0) (at 74.168 104.8766 0)
       (effects (font (size 1.27 1.27)) (justify left))
     )
@@
   (symbol (lib_id "Device:R") (at 87.63 62.865 0) (unit 1)
     (in_bom yes) (on_board yes)
-    (property "Reference" "R?" (id 0) (at 89.408 61.6966 0)
-      (effects (font (size 1.27 1.27)) (justify left))
-    )
-    (property "Value" "R" (id 1) (at 89.408 64.008 0)
+    (property "Reference" "R32" (id 0) (at 89.408 61.6966 0)
+      (effects (font (size 1.27 1.27)) (justify left))
+    )
+    (property "Value" "330" (id 1) (at 89.408 64.008 0)
       (effects (font (size 1.27 1.27)) (justify left))
     )
@@
       (effects (font (size 1.27 1.27)) (justify left))
     )
-    (property "Value" "R" (id 1) (at 89.408 151.638 0)
+    (property "Value" "330" (id 1) (at 89.408 151.638 0)
       (effects (font (size 1.27 1.27)) (justify left))
     )
@@
   (symbol (lib_id "Device:R") (at 158.75 83.185 180) (unit 1)
     (in_bom yes) (on_board yes)
-    (property "Reference" "R?" (id 0) (at 160.528 82.0166 0)
-      (effects (font (size 1.27 1.27)) (justify right))
-    )
-    (property "Value" "3.9k" (id 1) (at 160.528 84.328 0)
+    (property "Reference" "R36" (id 0) (at 160.528 82.0166 0)
+      (effects (font (size 1.27 1.27)) (justify right))
+    )
+    (property "Value" "9k" (id 1) (at 160.528 84.328 0)
       (effects (font (size 1.27 1.27)) (justify right))
     )
@@
   (symbol (lib_id "Device:R") (at 158.75 94.615 180) (unit 1)
     (in_bom yes) (on_board yes)
-    (property "Reference" "R?" (id 0) (at 160.528 93.4466 0)
-      (effects (font (size 1.27 1.27)) (justify right))
-    )
-    (property "Value" "3.9k" (id 1) (at 160.528 95.758 0)
+    (property "Reference" "R37" (id 0) (at 160.528 93.4466 0)
+      (effects (font (size 1.27 1.27)) (justify right))
+    )
+    (property "Value" "9k" (id 1) (at 160.528 95.758 0)
       (effects (font (size 1.27 1.27)) (justify right))
     )
@@
   (symbol (lib_id "Device:R") (at 177.8 89.535 270) (unit 1)
     (in_bom yes) (on_board yes)
-    (property "Reference" "R?" (id 0) (at 177.8 84.2772 90))
-    (property "Value" "3.9k" (id 1) (at 177.8 86.5886 90))
+    (property "Reference" "R35" (id 0) (at 177.8 84.2772 90))
+    (property "Value" "3k" (id 1) (at 177.8 86.5886 90))
     (property "Footprint" "" (id 2) (at 177.8 87.757 90)
       (effects (font (size 1.27 1.27)) hide)
@@
   (symbol (lib_id "Device:R") (at 201.93 95.885 180) (unit 1)
     (in_bom yes) (on_board yes)
-    (property "Reference" "R?" (id 0) (at 203.708 94.7166 0)
+    (property "Reference" "R34" (id 0) (at 203.708 94.7166 0)
       (effects (font (size 1.27 1.27)) (justify right))
     )
@@
   (symbol (lib_id "Diode:1N4148") (at 72.39 52.705 90) (unit 1)
     (in_bom yes) (on_board yes)
-    (property "Reference" "D?" (id 0) (at 74.3966 51.5366 90)
+    (property "Reference" "D31" (id 0) (at 74.3966 51.5366 90)
       (effects (font (size 1.27 1.27)) (justify right))
     )
@@
   (symbol (lib_id "Diode:1N4148") (at 72.39 65.405 90) (unit 1)
     (in_bom yes) (on_board yes)
-    (property "Reference" "D?" (id 0) (at 74.3966 64.2366 90)
+    (property "Reference" "D32" (id 0) (at 74.3966 64.2366 90)
       (effects (font (size 1.27 1.27)) (justify right))
     )
@@
   (symbol (lib_id "Diode:1N4148") (at 72.39 149.225 90) (unit 1)
     (in_bom yes) (on_board yes)
-    (property "Reference" "D?" (id 0) (at 74.3966 148.0566 90)
+    (property "Reference" "D33" (id 0) (at 74.3966 148.0566 90)
       (effects (font (size 1.27 1.27)) (justify right))
     )
@@
   (symbol (lib_id "Diode:1N4148") (at 72.39 159.385 90) (unit 1)
     (in_bom yes) (on_board yes)
-    (property "Reference" "D?" (id 0) (at 74.3966 158.2166 90)
+    (property "Reference" "D34" (id 0) (at 74.3966 158.2166 90)
       (effects (font (size 1.27 1.27)) (justify right))
     )
@@
   (symbol (lib_id "Diode:1N4148") (at 120.65 99.695 90) (unit 1)
     (in_bom yes) (on_board yes)
-    (property "Reference" "D?" (id 0) (at 122.6566 98.5266 90)
+    (property "Reference" "D35" (id 0) (at 122.6566 98.5266 90)
       (effects (font (size 1.27 1.27)) (justify right))
     )
@@
   (symbol (lib_id "Diode:1N4148") (at 120.65 112.395 90) (unit 1)
     (in_bom yes) (on_board yes)
-    (property "Reference" "D?" (id 0) (at 122.6566 111.2266 90)
+    (property "Reference" "D36" (id 0) (at 122.6566 111.2266 90)
       (effects (font (size 1.27 1.27)) (justify right))
     )
@@
   (symbol (lib_id "Diode:1N4148") (at 135.89 99.695 90) (unit 1)
     (in_bom yes) (on_board yes)
-    (property "Reference" "D?" (id 0) (at 137.8966 98.5266 90)
+    (property "Reference" "D37" (id 0) (at 137.8966 98.5266 90)
       (effects (font (size 1.27 1.27)) (justify right))
     )
@@
   (symbol (lib_id "Diode:1N4148") (at 135.89 112.395 90) (unit 1)
     (in_bom yes) (on_board yes)
-    (property "Reference" "D?" (id 0) (at 137.8966 111.2266 90)
+    (property "Reference" "D38" (id 0) (at 137.8966 111.2266 90)
       (effects (font (size 1.27 1.27)) (justify right))
     )
@@
   (symbol (lib_id "Device:C") (at 152.4 118.745 0) (unit 1)
     (in_bom yes) (on_board yes)
-    (property "Reference" "C?" (id 0) (at 155.321 117.5766 0)
-      (effects (font (size 1.27 1.27)) (justify left))
-    )
-    (property "Value" "100n" (id 1) (at 155.321 119.888 0)
+    (property "Reference" "C31" (id 0) (at 155.321 117.5766 0)
+      (effects (font (size 1.27 1.27)) (justify left))
+    )
+    (property "Value" "1.5n" (id 1) (at 155.321 119.888 0)
       (effects (font (size 1.27 1.27)) (justify left))
     )
@@
   (symbol (lib_id "Transistor_BJT:MMBT3906") (at 85.09 75.565 0) (mirror x) (unit 1)
     (in_bom yes) (on_board yes)
-    (property "Reference" "Q?" (id 0) (at 89.9414 74.3966 0)
+    (property "Reference" "Q31" (id 0) (at 89.9414 74.3966 0)
       (effects (font (size 1.27 1.27)) (justify left))
     )
@@
   (symbol (lib_id "Transistor_BJT:MMBT3904") (at 85.09 135.255 0) (unit 1)
     (in_bom yes) (on_board yes)
-    (property "Reference" "Q?" (id 0) (at 89.9414 134.0866 0)
+    (property "Reference" "Q32" (id 0) (at 89.9414 134.0866 0)
       (effects (font (size 1.27 1.27)) (justify left))
     )
@@
   (symbol (lib_id "Class_D_Amplfier_v2-rescue:LM319-Comparator") (at 177.8 103.505 0) (unit 1)
     (in_bom yes) (on_board yes)
-    (property "Reference" "U?" (id 0) (at 177.8 94.1832 0))
+    (property "Reference" "U31" (id 0) (at 177.8 94.1832 0))
     (property "Value" "LM319" (id 1) (at 177.8 96.4946 0))
     (property "Footprint" "" (id 2) (at 177.8 103.505 0)
@@
     (pin "5")
   )
-  (symbol (lib_id "Class_D_Amplfier_v2-rescue:LM319-Comparator") (at 182.245 136.525 0) (unit 1)
-    (in_bom yes) (on_board yes)
-    (property "Reference" "U?" (id 0) (at 182.245 127.2032 0))
+  (symbol (lib_id "Class_D_Amplfier_v2-rescue:LM319-Comparator") (at 182.245 136.525 0) (unit 2)
+    (in_bom yes) (on_board yes)
+    (property "Reference" "U31" (id 0) (at 182.245 127.2032 0))
     (property "Value" "LM319" (id 1) (at 182.245 129.5146 0))
     (property "Footprint" "" (id 2) (at 182.245 136.525 0)
@@
       (effects (font (size 1.27 1.27)) hide)
     )
-    (pin "1")
-    (pin "12")
-    (pin "2")
-    (pin "3")
-    (pin "4")
-    (pin "5")
+    (pin "10")
+    (pin "13")
+    (pin "14")
+    (pin "7")
+    (pin "8")
+    (pin "9")
   )
 )
